File: Hardware/LampeSolaire2.kicad_pcb (KiCad board)
At the start: 2 copper layers, 100 x 17.5 mm, 29 parts, among them J1 Connector, J2 CONN_ICSP, J3 Leds, J4 Led 2, P1 GREEN, P2 LED, P3 LED, P4 RED, P5 GREEN, U1 RF_RECEIVER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

Commit message: Nouvelle version
Other:
- net class Default removed
- net class Ground removed
- net class Led_LowResistance removed
