File: Hardware/LampeSolairePetite.kicad_pcb (KiCad board)
At the start: 2 copper layers, 62 x 21 mm, 24 parts, among them J1 CONN_ICSP, J2 Battery connector, J3 Connector_4p_r, J4 Connecteur LORA SX1278, P1 GREEN, P2 GREEN, P3 RED, P4 GREEN, U1 NCP114, U2 PIC16F1827

Commit message: Finished lampe
Parts:
- turned P1 to -90 degrees
- turned P2 to -90 degrees
- turned P3 to -90 degrees
- turned P4 to -90 degrees
Connections:
- net VCC_3V3 renamed +3V3
- P1 pad 1: GND -> Net-(R1-Pad2)
- P1 pad 2: Net-(P1-Pad2) -> GND
- P2 pad 1: LED_GREEN -> Net-(R3-Pad2)
- P2 pad 2: Net-(P2-Pad2) -> LED_GREEN
- P3 pad 1: LED_RED -> Net-(R4-Pad2)
- P3 pad 2: Net-(P3-Pad2) -> LED_RED
- P4 pad 1: BATTERY_IND -> Net-(R6-Pad2)
- P4 pad 2: Net-(P4-Pad2) -> BATTERY_IND
- R1 pad 2: Net-(P1-Pad2) -> Net-(R1-Pad2)
- R3 pad 2: Net-(P2-Pad2) -> Net-(R3-Pad2)
- R4 pad 2: Net-(P3-Pad2) -> Net-(R4-Pad2)
- R6 pad 2: Net-(P4-Pad2) -> Net-(R6-Pad2)
Routing:
- net Net-(R6-Pad2): track 0.00 -> 2.29 mm
- net Net-(P4-Pad2): track 2.29 -> 0.00 mm
- net Net-(R1-Pad2): track 0.00 -> 2.24 mm
- net Net-(P1-Pad2): track 2.24 -> 0.00 mm
- net Net-(R4-Pad2): track 0.00 -> 2.24 mm
- net Net-(P3-Pad2): track 2.24 -> 0.00 mm
- net Net-(R3-Pad2): track 0.00 -> 2.19 mm
- net Net-(P2-Pad2): track 2.19 -> 0.00 mm
